Commit message: include joints limits in exoter odometry urdf file

File: data/odometry/exoter_odometry_model.urdf (robot description, URDF)
Before this commit: robot exoter, 26 links, 25 joints
Joints:
- joint 00_joint: limit (none) -> lower=-1.6 upper=1.6 effort=100 velocity=6.28
- joint 01_joint: limit (none) -> lower=-1.6 upper=1.6 effort=100 velocity=6.28
- joint 02_joint: limit (none) -> lower=-1.6 upper=1.6 effort=100 velocity=6.28
- joint 0_0_joint: limit (none) -> lower=-1.6 upper=1.6 effort=100 velocity=6.28
- joint 0_1_joint: limit (none) -> lower=-1.6 upper=1.6 effort=100 velocity=6.28
- joint 0_2_joint: limit (none) -> lower=-1.6 upper=1.6 effort=100 velocity=6.28
- joint 0_3_joint: limit (none) -> lower=-1.6 upper=1.6 effort=100 velocity=6.28
- joint 1_0_joint: limit (none) -> lower=-1.6 upper=1.6 effort=100 velocity=6.28
- joint 1_1_joint: limit (none) -> lower=-1.6 upper=1.6 effort=100 velocity=6.28
- joint 1_2_joint: limit (none) -> lower=-1.6 upper=1.6 effort=100 velocity=6.28
- joint 1_3_joint: limit (none) -> lower=-1.6 upper=1.6 effort=100 velocity=6.28
- joint 2_0_joint: limit (none) -> lower=-1.6 upper=1.6 effort=100 velocity=6.28
- joint 2_1_joint: limit (none) -> lower=-1.6 upper=1.6 effort=100 velocity=6.28
- joint 2_2_joint: limit (none) -> lower=-1.6 upper=1.6 effort=100 velocity=6.28
- joint 3_0_joint: limit (none) -> lower=-1.6 upper=1.6 effort=100 velocity=6.28
- joint 3_1_joint: limit (none) -> lower=-1.6 upper=1.6 effort=100 velocity=6.28
- joint 3_2_joint: limit (none) -> lower=-1.6 upper=1.6 effort=100 velocity=6.28
- joint 4_0_joint: limit (none) -> lower=-1.6 upper=1.6 effort=100 velocity=6.28
- joint 4_1_joint: limit (none) -> lower=-1.6 upper=1.6 effort=100 velocity=6.28
- joint 4_2_joint: limit (none) -> lower=-1.6 upper=1.6 effort=100 velocity=6.28
- joint 4_3_joint: limit (none) -> lower=-1.6 upper=1.6 effort=100 velocity=6.28
- joint 5_0_joint: limit (none) -> lower=-1.6 upper=1.6 effort=100 velocity=6.28
- joint 5_1_joint: limit (none) -> lower=-1.6 upper=1.6 effort=100 velocity=6.28
- joint 5_2_joint: limit (none) -> lower=-1.6 upper=1.6 effort=100 velocity=6.28
- joint 5_3_joint: limit (none) -> lower=-1.6 upper=1.6 effort=100 velocity=6.28
