Commit message: added new URDF file to use with three_odometry configuration file for threed_odometry task new ruby scripts to process logs and compare different odometries

File: data/odometry/exoter_odometry_model_complete.urdf (robot description, URDF)
Before this commit: robot exoter, 56 links, 55 joints
Joints:
- joint fl_drive: limit lower=-3.14 upper=3.14 effort=100 velocity=6.28 -> lower=-3.14 upper=3.14 effort=100 velocity=60.28
- joint fl_translation: limit lower=-3.14 upper=3.14 effort=100 velocity=6.28 -> lower=-3.14 upper=3.14 effort=100 velocity=10.00
- joint fr_drive: limit lower=-3.14 upper=3.14 effort=100 velocity=6.28 -> lower=-3.14 upper=3.14 effort=100 velocity=60.28
- joint fr_translation: limit lower=-3.14 upper=3.14 effort=100 velocity=6.28 -> lower=-3.14 upper=3.14 effort=100 velocity=10.00
- joint ml_drive: limit lower=-3.14 upper=3.14 effort=100 velocity=6.28 -> lower=-3.14 upper=3.14 effort=100 velocity=60.28
- joint ml_translation: limit lower=-3.14 upper=3.14 effort=100 velocity=6.28 -> lower=-3.14 upper=3.14 effort=100 velocity=10.00
- joint mr_drive: limit lower=-3.14 upper=3.14 effort=100 velocity=6.28 -> lower=-3.14 upper=3.14 effort=100 velocity=60.28
- joint mr_translation: limit lower=-3.14 upper=3.14 effort=100 velocity=6.28 -> lower=-3.14 upper=3.14 effort=100 velocity=10.00
- joint rl_drive: limit lower=-3.14 upper=3.14 effort=100 velocity=6.28 -> lower=-3.14 upper=3.14 effort=100 velocity=60.28
- joint rl_translation: limit lower=-3.14 upper=3.14 effort=100 velocity=6.28 -> lower=-3.14 upper=3.14 effort=100 velocity=10.00
- joint rr_drive: limit lower=-3.14 upper=3.14 effort=100 velocity=6.28 -> lower=-3.14 upper=3.14 effort=100 velocity=60.28
- joint rr_translation: limit lower=-3.14 upper=3.14 effort=100 velocity=6.28 -> lower=-3.14 upper=3.14 effort=100 velocity=10.00
