Commit message: add limits in exoter urdf in order to display with the new version of rock-roboviz command

File: data/urdf/exoter.urdf (robot description, URDF)
Before this commit: robot exoter, 30 links, 29 joints
Joints:
- joint fl_drive: limit (none) -> lower=-3.14 upper=3.14 effort=100 velocity=6.28
- joint fl_mimic: limit (none) -> lower=-1.6 upper=1.6 effort=100 velocity=6.28
- joint fl_steer: limit (none) -> lower=-1.6 upper=1.6 effort=100 velocity=6.28
- joint fl_walking: limit (none) -> lower=-1.6 upper=1.6 effort=100 velocity=6.28
- joint fr_drive: limit (none) -> lower=-3.14 upper=3.14 effort=100 velocity=6.28
- joint fr_mimic: limit (none) -> lower=-1.6 upper=1.6 effort=100 velocity=6.28
- joint fr_steer: limit (none) -> lower=-1.6 upper=1.6 effort=100 velocity=6.28
- joint fr_walking: limit (none) -> lower=-1.6 upper=1.6 effort=100 velocity=6.28
- joint left_passive: limit (none) -> lower=-1.6 upper=1.6 effort=100 velocity=6.28
- joint mast_joint: limit (none) -> lower=-1.6 upper=1.6 effort=100 velocity=6.28
- joint mast_top_joint: limit (none) -> lower=-1.6 upper=1.6 effort=100 velocity=6.28
- joint ml_drive: limit (none) -> lower=-3.14 upper=3.14 effort=100 velocity=6.28
- joint ml_mimic: limit (none) -> lower=-1.6 upper=1.6 effort=100 velocity=6.28
- joint ml_walking: limit (none) -> lower=-1.6 upper=1.6 effort=100 velocity=6.28
- joint mr_drive: limit (none) -> lower=-3.14 upper=3.14 effort=100 velocity=6.28
- joint mr_mimic: limit (none) -> lower=-1.6 upper=1.6 effort=100 velocity=6.28
- joint mr_walking: limit (none) -> lower=-1.6 upper=1.6 effort=100 velocity=6.28
- joint pan_joint: limit (none) -> lower=-1.6 upper=1.6 effort=100 velocity=6.28
- joint rear_passive: limit (none) -> lower=-1.6 upper=1.6 effort=100 velocity=6.28
- joint right_passive: limit (none) -> lower=-1.6 upper=1.6 effort=100 velocity=6.28
- joint rl_drive: limit (none) -> lower=-3.14 upper=3.14 effort=100 velocity=6.28
- joint rl_mimic: limit (none) -> lower=-1.6 upper=1.6 effort=100 velocity=6.28
- joint rl_steer: limit (none) -> lower=-1.6 upper=1.6 effort=100 velocity=6.28
- joint rl_walking: limit (none) -> lower=-1.6 upper=1.6 effort=100 velocity=6.28
- joint rr_drive: limit (none) -> lower=-3.14 upper=3.14 effort=100 velocity=6.28
- joint rr_mimic: limit (none) -> lower=-1.6 upper=1.6 effort=100 velocity=6.28
- joint rr_steer: limit (none) -> lower=-1.6 upper=1.6 effort=100 velocity=6.28
- joint rr_walking: limit (none) -> lower=-1.6 upper=1.6 effort=100 velocity=6.28
- joint tilt_joint: limit (none) -> lower=-1.6 upper=1.6 effort=100 velocity=6.28

Commit message: urdf/exoter: rename root frame to body to make it work with the current robot visualization plugin

File: data/urdf/exoter.urdf (robot description, URDF)
Before this commit: robot exoter, 30 links, 29 joints
Links:
- removed link body_base
- added link body; visual mesh filename=./meshes/exoter/body_base_vicon_and_gps.stl scale=1 1 1
Joints:
- joint left_passive: parent body_base -> body
- joint mast_joint: parent body_base -> body
- joint rear_passive: parent body_base -> body
- joint right_passive: parent body_base -> body
